File: KiCAD/Phase_shifter/Phase_shifter.kicad_sch (KiCad schematic)
At the start: 6 parts

Commit message: a
Parts:
- C1, C2: footprint (none) -> Capacitor_SMD:C_0603_1608Metric_Pad1.08x0.95mm_HandSolder
- J1, J2: footprint (none) -> Phase_shifter:Connector
- R1: footprint (none) -> Resistor_SMD:R_0603_1608Metric_Pad0.98x0.95mm_HandSolder
- U1: footprint (none) -> Phase_shifter:MAPS-010144
Connections:
- net GND: now also J1.2 (SHIELD), J2.2 (SHIELD); no longer J1. (SHIELD), J2. (SHIELD)
- net RF_OUT: now reaches U1.14 (RF_OUT)
- net RF_OUT: now also J2.1 (COAX); no longer J2. (SHIELD)
- net RF_IN: now reaches U1.5 (RF_IN)
- net RF_IN: now also J1.1 (COAX); no longer J1. (SHIELD)
Changed lines of the file:
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@@
+		)
+	)
+	(label "RF_IN"
+		(at 114.3 105.41 0)
+		(effects
+			(font
+				(size 1.27 1.27)
+			)
+			(justify left bottom)
 		)
 	)
@@
 		)
 	)
-	(symbol
-		(lib_name "COAX_CON_1")
+	(label "RF_OUT"
+		(at 160.02 105.41 0)
+		(effects
+			(font
+				(size 1.27 1.27)
+			)
+			(justify left bottom)
+		)
+	)
+	(symbol
 		(lib_id "Phase_shifter:COAX_CON")
 		(at 182.88 106.68 0)
@@
 			)
 		)
-		(property "Footprint" ""
+		(property "Footprint" "Phase_shifter:Connector"
 			(at 182.88 106.68 0)
 			(effects
@@
 			)
 		)
-		(pin ""
-		)
-		(pin ""
+		(pin "1"
+		)
+		(pin "2"
 		)
 		(instances
@@
 			)
 		)
-		(property "Footprint" ""
+		(property "Footprint" "Phase_shifter:Connector"
 			(at 96.52 106.68 0)
 			(effects
@@
 			)
 		)
-		(pin ""
-		)
-		(pin ""
+		(pin "2"
+		)
+		(pin "1"
 		)
 		(instances
@@
 			)
 		)
-		(property "Footprint" ""
+		(property "Footprint" "Phase_shifter:MAPS-010144"
 			(at 139.7 101.6 0)
 			(effects
@@
 			)
 		)
-		(property "Footprint" ""
+		(property "Footprint" "Resistor_SMD:R_0603_1608Metric_Pad0.98x0.95mm_HandSolder"
 			(at 117.602 88.9 90)
 			(effects
@@
 			)
 		)
-		(property "Footprint" ""
+		(property "Footprint" "Capacitor_SMD:C_0603_1608Metric_Pad1.08x0.95mm_HandSolder"
 			(at 166.0652 116.84 0)
 			(effects
@@
 			)
 		)
-		(property "Footprint" ""
+		(property "Footprint" "Capacitor_SMD:C_0603_1608Metric_Pad1.08x0.95mm_HandSolder"
 			(at 112.7252 115.57 0)
 			(effects
