File: KiCAD/Phase_shifter_test_board/Phase_shifter_test_board/Phase_shifter_test_board.kicad_pcb (KiCad board)
At the start: 2 copper layers, 30.5 x 25.2 mm, 7 parts, among them J3 Conn_01x10_Pin

Commit message: phase shifter
Parts:
- added J4: ~, Phase_shifter:Conn, F.Cu at (117.0, 114.8)
- added J5: Conn_02x05_Odd_Even, Connector_PinHeader_2.54mm:PinHeader_2x05_P2.54mm_Vertical, F.Cu at (104.5, 89.0)
- added R2: R, Resistor_SMD:R_0603_1608Metric_Pad0.98x0.95mm_HandSolder, F.Cu at (104.9, 81.2)
- added R3: R, Resistor_SMD:R_0603_1608Metric_Pad0.98x0.95mm_HandSolder, F.Cu at (107.4, 83.4)
- added R4: R, Resistor_SMD:R_0603_1608Metric_Pad0.98x0.95mm_HandSolder, F.Cu at (111.8, 83.4)
- added R5: R, Resistor_SMD:R_0603_1608Metric_Pad0.98x0.95mm_HandSolder, F.Cu at (114.3, 81.2)
- added R6: R, Resistor_SMD:R_0603_1608Metric_Pad0.98x0.95mm_HandSolder, F.Cu at (101.8, 82.4)
- added R7: R, Resistor_SMD:R_0603_1608Metric_Pad0.98x0.95mm_HandSolder, F.Cu at (104.4, 91.6)
- added SW1: SW_DIP_x04, Button_Switch_THT:SW_DIP_SPSTx04_Slide_9.78x12.34mm_W7.62mm_P2.54mm, F.Cu at (105.8, 78.4)
- J3: value Conn_01x10_Pin -> ~; footprint Connector_PinHeader_2.54mm:PinHeader_1x10_P2.54mm_Vertical_SMD_Pin1Left -> Phase_shifter:Conn
- moved J3 56.8 mm to (103.1, 114.8)
- moved J2 46.1 mm to (117.0, 101.0)
- moved C2 43.4 mm to (113.0, 96.0), turned to 90 degrees
- moved U1 40.7 mm to (110.0, 100.2)
- moved C1 39.3 mm to (107.2, 96.0), turned to 90 degrees
- moved R1 38.6 mm to (104.4, 93.0), turned to 0 degrees
- moved J1 35.2 mm to (103.1, 101.0)
Connections:
- J3 pad 1: GND -> /RF REF
- J3 pad 2: VCC -> GND
- U1 pad 22: /LE -> /LE / D3
- U1 pad 23: /CLK -> /CLK / D2
- U1 pad 24: /SER IN -> /SER IN / D1
Routing:
- net /LE / D3: track 0.00 -> 22.5 mm
- net Net-(R6-Pad1): track 0.00 -> 20.0 mm
- net /RF REF: track 0.00 -> 15.6 mm
- net VCC: track 48.1 -> 32.9 mm, vias 0 -> 1
- net /D4: track 9.30 -> 22.3 mm
- net /SER IN / D1: track 0.00 -> 12.5 mm
- net /SER IN: track 12.4 -> 0.00 mm
- net /LE: track 11.8 -> 0.00 mm
- net /D6: track 11.8 -> 23.1 mm
- net /CLK / D2: track 0.00 -> 9.37 mm
- net GND: track 22.4 -> 31.5 mm, vias 0 -> 11
- net /D5: track 13.5 -> 21.9 mm
- net /CLK: track 8.28 -> 0.00 mm
- net /RF IN: track 9.20 -> 4.65 mm
- net /RF OUT: track 9.20 -> 4.65 mm
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- added copper zone on F.Cu, net /RF REF
- removed copper zone on F.Cu, net GND
Other:
- board size 30.5 x 25.2 mm -> 19.5 x 54.2 mm

Commit message: test board
Parts:
- removed R1, R6: R, Resistor_SMD:R_0603_1608Metric_Pad0.98x0.95mm_HandSolder
- added C3: C, Capacitor_SMD:C_0603_1608Metric_Pad1.08x0.95mm_HandSolder, F.Cu at (104.8, 101.0)
- added C4: C, Capacitor_SMD:C_0603_1608Metric_Pad1.08x0.95mm_HandSolder, F.Cu at (115.2, 101.0)
- added H1: MountingHole, MountingHole:MountingHole_3.2mm_M3, F.Cu at (103.7, 66.5)
- added H2: MountingHole, MountingHole:MountingHole_3.2mm_M3, F.Cu at (116.1, 66.6)
- added H3: MountingHole, MountingHole:MountingHole_3.2mm_M3, F.Cu at (103.5, 125.4)
- added H4: MountingHole, MountingHole:MountingHole_3.2mm_M3, F.Cu at (116.5, 125.4)
- added J6: Conn_01x02_Pin, Connector_PinHeader_2.54mm:PinHeader_1x02_P2.54mm_Vertical, F.Cu at (102.7, 86.0)
- moved R2 9.71 mm to (109.0, 90.0), turned to 90 degrees
- moved R5 9.07 mm to (116.5, 90.0), turned to 90 degrees
- moved R3 7.76 mm to (111.5, 90.0), turned to 90 degrees
- moved R4 6.96 mm to (114.0, 90.0), turned to 90 degrees
- moved J5 3.69 mm to (106.6, 85.9)
- moved SW1 2.47 mm to (108.0, 79.6)
- moved R7 1.64 mm to (104.8, 90.0), turned to 90 degrees
- moved C1 0.25 mm to (107.5, 96.0)
- moved C2 0.25 mm to (112.8, 96.0)
Connections:
- SW1 pad 5: Net-(R6-Pad1) -> VCC
- SW1 pad 6: Net-(R6-Pad1) -> VCC
- SW1 pad 7: Net-(R6-Pad1) -> VCC
- SW1 pad 8: Net-(R6-Pad1) -> VCC
- U1 pad 14: /RF OUT -> Net-(U1-RF_OUT)
- U1 pad 5: /RF IN -> Net-(U1-RF_IN)
Routing:
- net VCC: track 32.9 -> 59.5 mm
- net Net-(R6-Pad1): track 20.0 -> 0.00 mm
- net GND: track 31.5 -> 12.3 mm, vias 11 -> 183
- net /P/S: track 10.5 -> 16.0 mm
- net /SER OUT: track 15.8 -> 20.5 mm
- net VEE: track 11.4 -> 15.5 mm, vias 0 -> 1
- net /CLK / D2: track 9.37 -> 13.4 mm
- net /SER IN / D1: track 12.5 -> 15.7 mm
- net /RF IN: track 4.65 -> 1.59 mm
- net /RF OUT: track 4.65 -> 1.59 mm
- net Net-(U1-RF_IN): track 0.00 -> 1.19 mm
- net Net-(U1-RF_OUT): track 0.00 -> 1.10 mm
- net /LE / D3: track 22.5 -> 21.9 mm, vias 0 -> 2
- added copper zone on F.Cu, net GND
- added copper zone on F.Cu, net Net-(U1-RF_IN)
- added copper zone on F.Cu, net Net-(U1-RF_OUT)
Other:
- board size 19.5 x 54.2 mm -> 19.5 x 65.2 mm

Commit message: skeleton
Changed lines of the file:
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@@
 		(allow_soldermask_bridges_in_footprints no)
 		(pcbplotparams
-			(layerselection 0x0001080_ffffffff)
+			(layerselection 0x0001000_ffffffff)
 			(plot_on_all_layers_selection 0x0000000_00000000)
 			(disableapertmacros no)
@@
 			(at 0 -4.2 0)
 			(layer "F.SilkS")
+			(hide yes)
 			(effects
 				(font
@@
 			(at 0 -4.2 0)
 			(layer "F.SilkS")
+			(hide yes)
 			(effects
 				(font
@@
 			)
 		)
+	)
+	(zone
+		(net 0)
+		(net_name "")
+		(layers "F&B.Cu")
+		(hatch edge 0.5)
+		(connect_pads
+			(clearance 0)
+		)
+		(min_thickness 0.25)
+		(filled_areas_thickness no)
+		(keepout
+			(tracks not_allowed)
+			(vias not_allowed)
+			(pads not_allowed)
+			(copperpour not_allowed)
+			(footprints allowed)
+		)
+		(fill
+			(thermal_gap 0.5)
+			(thermal_bridge_width 0.5)
+		)
+		(polygon
+			(pts
+				(xy 106 125.375) (xy 105.980287 125.061667) (xy 105.921458 124.753275) (xy 105.824441 124.454689)
+				(xy 105.690767 124.170616) (xy 105.522542 123.905537) (xy 105.322422 123.663632) (xy 105.09356 123.448717)
+				(xy 104.839567 123.26418) (xy 104.564448 123.112932) (xy 104.272542 122.997359) (xy 103.968453 122.919282)
+				(xy 103.656976 122.879933) (xy 103.343024 122.879933) (xy 103.031547 122.919282) (xy 102.727458 122.997359)
+				(xy 102.435552 123.112932) (xy 102.160433 123.26418) (xy 101.90644 123.448717) (xy 101.677578 123.663632)
+				(xy 101.477458 123.905537) (xy 101.309233 124.170616) (xy 101.175559 124.454689) (xy 101.078542 124.753275)
+				(xy 101.019713 125.061667) (xy 101 125.375) (xy 101.019713 125.688333) (xy 101.078542 125.996725)
+				(xy 101.175559 126.295311) (xy 101.309233 126.579384) (xy 101.477458 126.844463) (xy 101.677578 127.086368)
+				(xy 101.90644 127.301283) (xy 102.160433 127.48582) (xy 102.435552 127.637068) (xy 102.727458 127.752641)
+				(xy 103.031547 127.830718) (xy 103.343024 127.870067) (xy 103.656976 127.870067) (xy 103.968453 127.830718)
+				(xy 104.272542 127.752641) (xy 104.564448 127.637068) (xy 104.839567 127.48582) (xy 105.09356 127.301283)
+				(xy 105.322422 127.086368) (xy 105.522542 126.844463) (xy 105.690767 126.579384) (xy 105.824441 126.295311)
+				(xy 105.921458 125.996725) (xy 105.980287 125.688333) (xy 106 125.375)
+			)
+		)
+	)
+	(zone
+		(net 0)
+		(net_name "")
+		(layers "F&B.Cu")
+		(hatch edge 0.5)
+		(connect_pads
+			(clearance 0)
+		)
+		(min_thickness 0.25)
+		(filled_areas_thickness no)
+		(keepout
+			(tracks not_allowed)
+			(vias not_allowed)
+			(pads not_allowed)
+			(copperpour not_allowed)
+			(footprints allowed)
+		)
+		(fill
+			(thermal_gap 0.5)
+			(thermal_bridge_width 0.5)
+		)
+		(polygon
+			(pts
+				(xy 106.225 66.525) (xy 106.205287 66.211667) (xy 106.146458 65.903275) (xy 106.049441 65.604689)
+				(xy 105.915767 65.320616) (xy 105.747542 65.055537) (xy 105.547422 64.813632) (xy 105.31856 64.598717)
+				(xy 105.064567 64.41418) (xy 104.789448 64.262932) (xy 104.497542 64.147359) (xy 104.193453 64.069282)
+				(xy 103.881976 64.029933) (xy 103.568024 64.029933) (xy 103.256547 64.069282) (xy 102.952458 64.147359)
+				(xy 102.660552 64.262932) (xy 102.385433 64.41418) (xy 102.13144 64.598717) (xy 101.902578 64.813632)
+				(xy 101.702458 65.055537) (xy 101.534233 65.320616) (xy 101.400559 65.604689) (xy 101.303542 65.903275)
+				(xy 101.244713 66.211667) (xy 101.225 66.525) (xy 101.244713 66.838333) (xy 101.303542 67.146725)
+				(xy 101.400559 67.445311) (xy 101.534233 67.729384) (xy 101.702458 67.994463) (xy 101.902578 68.236368)
+				(xy 102.13144 68.451283) (xy 102.385433 68.63582) (xy 102.660552 68.787068) (xy 102.952458 68.902641)
+				(xy 103.256547 68.980718) (xy 103.568024 69.020067) (xy 103.881976 69.020067) (xy 104.193453 68.980718)
+				(xy 104.497542 68.902641) (xy 104.789448 68.787068) (xy 105.064567 68.63582) (xy 105.31856 68.451283)
+				(xy 105.547422 68.236368) (xy 105.747542 67.994463) (xy 105.915767 67.729384) (xy 106.049441 67.445311)
+				(xy 106.146458 67.146725) (xy 106.205287 66.838333) (xy 106.225 66.525)
+			)
+		)
+	)
+	(zone
+		(net 0)
+		(net_name "")
+		(layers "F&B.Cu")
+		(hatch edge 0.5)
+		(connect_pads
+			(clearance 0)
+		)
+		(min_thickness 0.25)
+		(filled_areas_thickness no)
+		(keepout
+			(tracks not_allowed)
+			(vias not_allowed)
+			(pads not_allowed)
+			(copperpour not_allowed)
+			(footprints allowed)
+		)
+		(fill
+			(thermal_gap 0.5)
+			(thermal_bridge_width 0.5)
+		)
+		(polygon
+			(pts
+				(xy 119 125.375) (xy 118.980287 125.061667) (xy 118.921458 124.753275) (xy 118.824441 124.454689)
+				(xy 118.690767 124.170616) (xy 118.522542 123.905537) (xy 118.322422 123.663632) (xy 118.09356 123.448717)
+				(xy 117.839567 123.26418) (xy 117.564448 123.112932) (xy 117.272542 122.997359) (xy 116.968453 122.919282)
+				(xy 116.656976 122.879933) (xy 116.343024 122.879933) (xy 116.031547 122.919282) (xy 115.727458 122.997359)
+				(xy 115.435552 123.112932) (xy 115.160433 123.26418) (xy 114.90644 123.448717) (xy 114.677578 123.663632)
+				(xy 114.477458 123.905537) (xy 114.309233 124.170616) (xy 114.175559 124.454689) (xy 114.078542 124.753275)
+				(xy 114.019713 125.061667) (xy 114 125.375) (xy 114.019713 125.688333) (xy 114.078542 125.996725)
+				(xy 114.175559 126.295311) (xy 114.309233 126.579384) (xy 114.477458 126.844463) (xy 114.677578 127.086368)
+				(xy 114.90644 127.301283) (xy 115.160433 127.48582) (xy 115.435552 127.637068) (xy 115.727458 127.752641)
+				(xy 116.031547 127.830718) (xy 116.343024 127.870067) (xy 116.656976 127.870067) (xy 116.968453 127.830718)
+				(xy 117.272542 127.752641) (xy 117.564448 127.637068) (xy 117.839567 127.48582) (xy 118.09356 127.301283)
+				(xy 118.322422 127.086368) (xy 118.522542 126.844463) (xy 118.690767 126.579384) (xy 118.824441 126.295311)
+				(xy 118.921458 125.996725) (xy 118.980287 125.688333) (xy 119 125.375)
+			)
+		)
+	)
+	(zone
+		(net 0)
+		(net_name "")
+		(layers "F&B.Cu")
+		(hatch edge 0.5)
+		(connect_pads
+			(clearance 0)
+		)
+		(min_thickness 0.25)
+		(filled_areas_thickness no)
+		(keepout
+			(tracks not_allowed)
+			(vias not_allowed)
+			(pads not_allowed)
+			(copperpour not_allowed)
+			(footprints allowed)
+		)
+		(fill
+			(thermal_gap 0.5)
+			(thermal_bridge_width 0.5)
+		)
+		(polygon
+			(pts
+				(xy 118.575 66.6) (xy 118.555287 66.286667) (xy 118.496458 65.978275) (xy 118.399441 65.679689)
+				(xy 118.265767 65.395616) (xy 118.097542 65.130537) (xy 117.897422 64.888632) (xy 117.66856 64.673717)
+				(xy 117.414567 64.48918) (xy 117.139448 64.337932) (xy 116.847542 64.222359) (xy 116.543453 64.144282)
+				(xy 116.231976 64.104933) (xy 115.918024 64.104933) (xy 115.606547 64.144282) (xy 115.302458 64.222359)
+				(xy 115.010552 64.337932) (xy 114.735433 64.48918) (xy 114.48144 64.673717) (xy 114.252578 64.888632)
+				(xy 114.052458 65.130537) (xy 113.884233 65.395616) (xy 113.750559 65.679689) (xy 113.653542 65.978275)
+				(xy 113.594713 66.286667) (xy 113.575 66.6) (xy 113.594713 66.913333) (xy 113.653542 67.221725)
+				(xy 113.750559 67.520311) (xy 113.884233 67.804384) (xy 114.052458 68.069463) (xy 114.252578 68.311368)
+				(xy 114.48144 68.526283) (xy 114.735433 68.71082) (xy 115.010552 68.862068) (xy 115.302458 68.977641)
+				(xy 115.606547 69.055718) (xy 115.918024 69.095067) (xy 116.231976 69.095067) (xy 116.543453 69.055718)
+				(xy 116.847542 68.977641) (xy 117.139448 68.862068) (xy 117.414567 68.71082) (xy 117.66856 68.526283)
+				(xy 117.897422 68.311368) (xy 118.097542 68.069463) (xy 118.265767 67.804384) (xy 118.399441 67.520311)
+				(xy 118.496458 67.221725) (xy 118.555287 66.913333) (xy 118.575 66.6)
+			)
+		)
